File: PCB/LimeShield/videobrick_alpha4.brd (EAGLE design)
At the start: 64.6 x 63.2 mm, 91 parts, among them CON1 A10_OLINUXINO_LIME_SHIELD_TEM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, K1 685119134923, Q1 BSS123, Q2 BSS123, Q3 BSS123, Q4 BSS123, U1 ADV7611BSWZ-P, U2 TPS72018DRVR, Y1 CRYSTAL_5_3.2

Commit message: version die bestellt wird
Parts:
- added TP1, TP2: TPTP06R, testpad:TP06R
- moved LOGO1 49.5 mm to (52.8, 21.9)
- moved C26 49.2 mm to (37.0, 30.0)
- moved C3 48.9 mm to (28.7, 34.2)
- moved C4 48.9 mm to (30.0, 34.2)
- moved D3 48.9 mm to (18.4, 34.5)
- moved C13 48.9 mm to (30.6, 28.1)
- moved C16 48.9 mm to (37.2, 35.8)
- moved C17 48.9 mm to (35.2, 32.3)
- moved C18 48.9 mm to (33.9, 32.3)
- moved C2 48.9 mm to (24.5, 40.4)
- moved C21 48.9 mm to (38.0, 26.9)
- moved C28 48.9 mm to (37.7, 23.6)
- moved C31 48.9 mm to (22.0, 43.9)
- moved C32 48.9 mm to (25.3, 15.5)
- moved C33 48.9 mm to (21.7, 15.5)
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Connections:
- removed net FMINL: CON1.4-19
- removed net FMINR: CON1.4-17
- removed net GNDA: CON1.1-4
- removed net HPCOM/HPCOMFB: CON1.1-16
- removed net HPOUTL: CON1.1-14
- removed net HPOUTR: CON1.1-18
- removed net I2S_DO0/AC97_DO/PB8/SATA-PWR-EN: CON1.3-16
- removed net I2S_DO2/PB10: CON1.3-18
- removed net I2S_DO3/PB11: CON1.3-20
- removed net IR0_RX/PB4: CON1.3-8
- removed net IR0_TX/SPDIF_MCLK/STANBYWFI/PB3: CON1.3-6
- removed net JTAG_CK0/SPI2_CLK/PB15: CON1.3-28
- removed net JTAG_DI0/SPI2_MISO/PB17: CON1.3-32
- removed net JTAG_DO0/SPI2_MOSI/PB16: CON1.3-30
- removed net JTAG_MS0/SPI2_CS0/PB14: CON1.3-26
- removed net LCD0_CLK/SMC_VCCEN/PD24: CON1.D-31
- removed net LCD0_D0/LVDS0_VP0/PD0: CON1.D-21
- removed net LCD0_D1/LVDS0_VN0/PD1: CON1.D-22
- removed net LCD0_D10/LVDS1_VP0/PD10: CON1.D-15
- removed net LCD0_D11/LVDS1_VN0/PD11: CON1.D-16
- removed net LCD0_D12/LVDS1_VP1/PD12: CON1.D-17
- removed net LCD0_D13/LVDS1_VN1/PD13: CON1.D-18
- removed net LCD0_D14/LVDS1_VP2/PD14: CON1.D-19
- removed net LCD0_D15/LVDS1_VN2/PD15: CON1.D-20
- removed net LCD0_D16/LVDS1_VPC/PD16: CON1.D-5
- removed net LCD0_D17/LVDS1_VNC/PD17: CON1.D-6
- removed net LCD0_D18/LVDS1_VP3/PD18: CON1.D-7
- removed net LCD0_D19/LVDS1_VN3/PD19: CON1.D-8
- removed net LCD0_D2/LVDS0_VP1/PD2: CON1.D-23
- removed net LCD0_D20/CSI1_MCLK/PD20: CON1.D-9
- removed net LCD0_D21/SMC_VPPEN/PD21: CON1.D-10
- removed net LCD0_D22/SMC_VPPPP/PD22: CON1.D-11
- removed net LCD0_D23/SMC_DET/PD23: CON1.D-12
- removed net LCD0_D3/LVDS0_VN1/PD3: CON1.D-24
- removed net LCD0_D4/LVDS0_VP2/PD4: CON1.D-25
- removed net LCD0_D5/LVDS0_VN2/PD5: CON1.D-26
- removed net LCD0_D6/LVDS0_VPC/PD6: CON1.D-27
- removed net LCD0_D7/LVDS0_VNC/PD7: CON1.D-28
- removed net LCD0_D8/LVDS0_VP3/PD8: CON1.D-13
- removed net LCD0_D9/LVDS0_VN3/PD9: CON1.D-14
- removed net LCD0_DE/SMC_RST/PD25: CON1.D-32
- removed net LCD0_HSYNC/SMC_SLK/PD26: CON1.D-29
- removed net LCD0_VSYNC/SMC_SDA/PD27: CON1.D-30
- removed net LCD1_CLK/ATACS1/KP_OUT4/SDC1_D0/CSI1_PCLK/PH24: CON1.3-34
- removed net LCD1_D7/ATAD3/UART5_RX/MS_CLK/EINT7/CSI1_D7/PH7/I2S_DO1/PB9/USB0-DRV: CON1.3-9
- removed net LCD1_HSYNC/ATAIOR/KP_OUT6/SDC1_D2/CSI1_HSYNC/PH26: CON1.3-38
- removed net LCD1_VSYNC/ATAIOW/KP_OUT7/SDC1_D3/CSI1_VSYNC/PH27: CON1.3-40
- removed net LRADC0: CON1.1-6
- removed net LRADC1: CON1.1-8
- removed net MIC1OUTN: CON1.4-8
- removed net MIC1OUTP: CON1.4-6
- removed net MICIN1: CON1.1-10
- removed net MICIN2: CON1.4-10
- removed net N$42: JP1.1
- removed net NC/IR0_RX/PB4: CON1.D-34
- removed net NC/IR0_TX/SPDIF_MCLK/STANBYWFI/PB3: CON1.D-33
- removed net NCE1/PC3/SATA-PWR-EN: CON1.1-29
- removed net NCE2/PC17: CON1.4-20
- removed net NCE3/PC18: CON1.1-31
- removed net NMI_N: CON1.4-4
- removed net NRB1/SDC2_CLK/PC7: CON1.4-16
- removed net NWP/PC16: CON1.4-18
- removed net RESET_N: CON1.3-5
- removed net SPI0_CS0/PC23: CON1.1-40
- removed net SPI2_CS1/SPDIF_DO/PB13: CON1.3-24
- removed net TVIN0: CON1.4-5
- removed net TVIN1: CON1.4-7
- removed net TVIN2: CON1.4-9
- removed net TVIN3: CON1.4-11
- removed net TVOUT0/VGA-G: CON1.1-20
- removed net TVOUT1/VGA-B: CON1.1-22
- removed net TVOUT2/VGA-R: CON1.1-24
- removed net TVOUT3: CON1.4-3
- removed net VMIC: CON1.1-12
- removed net XN_TP: CON1.D-38
- removed net XP_TP: CON1.D-37
- removed net YN_TP: CON1.D-40
- removed net YP_TP: CON1.D-39
- new net N$47: RN7.6, TP1.TP
- net CSI1_MLCK: now also TP2.TP
- net GND: now also JP1.1
Routing:
- net CSI1_PCLK: track 52.3 -> 47.7 mm
- net CSI1_MLCK: track 0.00 -> 2.61 mm, vias 0 -> 1
- net CVDD_1V8: track 37.1 -> 35.8 mm
- net N$47: track 0.00 -> 1.00 mm
- net DVDDIO_3V3: track 43.7 -> 44.5 mm
- net GND: vias 190 -> 189
