File: PCB/LimeShield/videobrick_alpha4.sch (EAGLE design)
At the start: 89 parts, among them CON1 A10_OLINUXINO_LIME_SHIELD_TEM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, K1 685119134923, Q1 BSS123, Q2 BSS123, Q3 BSS123, Q4 BSS123, U1 ADV7611BSWZ-P, U2 TPS72018DRVR, Y1 CRYSTAL_5_3.2

Commit message: a
Connections:
- new net LCD0_D4/LVDS0_VP2/PD4: CON1_LCD.25
- new net LCD0_D7/LVDS0_VNC/PD7: CON1_LCD.28
- new net LCD0_D8/LVDS0_VP3/PD8: CON1_LCD.13
- new net YN_TP: CON1_LCD.40
Other:
- moved on the sheet: C1, C10, C11, C12, C13, C14, C15, C16, C17, C18, C19, C2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

Commit message: version die bestellt wird
Parts:
- added TP1, TP2: TPTP06R, testpad:TPTP06R
Connections:
- removed net FMINL: CON1_GPIO-4.19
- removed net FMINR: CON1_GPIO-4.17
- removed net GNDA: CON1_GPIO-1.4
- removed net HPCOM/HPCOMFB: CON1_GPIO-1.16
- removed net HPOUTL: CON1_GPIO-1.14
- removed net HPOUTR: CON1_GPIO-1.18
- removed net I2S_DO0/AC97_DO/PB8/SATA-PWR-EN: CON1_GPIO-3.16
- removed net I2S_DO2/PB10: CON1_GPIO-3.18
- removed net I2S_DO3/PB11: CON1_GPIO-3.20
- removed net IR0_RX/PB4: CON1_GPIO-3.8
- removed net IR0_TX/SPDIF_MCLK/STANBYWFI/PB3: CON1_GPIO-3.6
- removed net JTAG_CK0/SPI2_CLK/PB15: CON1_GPIO-3.28
- removed net JTAG_DI0/SPI2_MISO/PB17: CON1_GPIO-3.32
- removed net JTAG_DO0/SPI2_MOSI/PB16: CON1_GPIO-3.30
- removed net JTAG_MS0/SPI2_CS0/PB14: CON1_GPIO-3.26
- removed net LCD0_CLK/SMC_VCCEN/PD24: CON1_LCD.31
- removed net LCD0_D0/LVDS0_VP0/PD0: CON1_LCD.21
- removed net LCD0_D1/LVDS0_VN0/PD1: CON1_LCD.22
- removed net LCD0_D10/LVDS1_VP0/PD10: CON1_LCD.15
- removed net LCD0_D11/LVDS1_VN0/PD11: CON1_LCD.16
- removed net LCD0_D12/LVDS1_VP1/PD12: CON1_LCD.17
- removed net LCD0_D13/LVDS1_VN1/PD13: CON1_LCD.18
- removed net LCD0_D14/LVDS1_VP2/PD14: CON1_LCD.19
- removed net LCD0_D15/LVDS1_VN2/PD15: CON1_LCD.20
- removed net LCD0_D16/LVDS1_VPC/PD16: CON1_LCD.5
- removed net LCD0_D17/LVDS1_VNC/PD17: CON1_LCD.6
- removed net LCD0_D18/LVDS1_VP3/PD18: CON1_LCD.7
- removed net LCD0_D19/LVDS1_VN3/PD19: CON1_LCD.8
- removed net LCD0_D2/LVDS0_VP1/PD2: CON1_LCD.23
- removed net LCD0_D20/CSI1_MCLK/PD20: CON1_LCD.9
- removed net LCD0_D21/SMC_VPPEN/PD21: CON1_LCD.10
- removed net LCD0_D22/SMC_VPPPP/PD22: CON1_LCD.11
- removed net LCD0_D23/SMC_DET/PD23: CON1_LCD.12
- removed net LCD0_D3/LVDS0_VN1/PD3: CON1_LCD.24
- removed net LCD0_D4/LVDS0_VP2/PD4: CON1_LCD.25
- removed net LCD0_D5/LVDS0_VN2/PD5: CON1_LCD.26
- removed net LCD0_D6/LVDS0_VPC/PD6: CON1_LCD.27
- removed net LCD0_D7/LVDS0_VNC/PD7: CON1_LCD.28
- removed net LCD0_D8/LVDS0_VP3/PD8: CON1_LCD.13
- removed net LCD0_D9/LVDS0_VN3/PD9: CON1_LCD.14
- removed net LCD0_DE/SMC_RST/PD25: CON1_LCD.32
- removed net LCD0_HSYNC/SMC_SLK/PD26: CON1_LCD.29
- removed net LCD0_VSYNC/SMC_SDA/PD27: CON1_LCD.30
- removed net LCD1_CLK/ATACS1/KP_OUT4/SDC1_D0/CSI1_PCLK/PH24: CON1_GPIO-3.34
- removed net LCD1_D7/ATAD3/UART5_RX/MS_CLK/EINT7/CSI1_D7/PH7/I2S_DO1/PB9/USB0-DRV: CON1_GPIO-3.9
- removed net LCD1_HSYNC/ATAIOR/KP_OUT6/SDC1_D2/CSI1_HSYNC/PH26: CON1_GPIO-3.38
- removed net LCD1_VSYNC/ATAIOW/KP_OUT7/SDC1_D3/CSI1_VSYNC/PH27: CON1_GPIO-3.40
- removed net LRADC0: CON1_GPIO-1.6
- removed net LRADC1: CON1_GPIO-1.8
- removed net MIC1OUTN: CON1_GPIO-4.8
- removed net MIC1OUTP: CON1_GPIO-4.6
- removed net MICIN1: CON1_GPIO-1.10
- removed net MICIN2: CON1_GPIO-4.10
- removed net N$42: JP1.1
- removed net NC/IR0_RX/PB4: CON1_LCD.34
- removed net NC/IR0_TX/SPDIF_MCLK/STANBYWFI/PB3: CON1_LCD.33
- removed net NCE1/PC3/SATA-PWR-EN: CON1_GPIO-1.29
- removed net NCE2/PC17: CON1_GPIO-4.20
- removed net NCE3/PC18: CON1_GPIO-1.31
- removed net NMI_N: CON1_GPIO-4.4
- removed net NRB1/SDC2_CLK/PC7: CON1_GPIO-4.16
- removed net NWP/PC16: CON1_GPIO-4.18
- removed net RESET_N: CON1_GPIO-3.5
- removed net SPI0_CS0/PC23: CON1_GPIO-1.40
- removed net SPI2_CS1/SPDIF_DO/PB13: CON1_GPIO-3.24
- removed net TVIN0: CON1_GPIO-4.5
- removed net TVIN1: CON1_GPIO-4.7
- removed net TVIN2: CON1_GPIO-4.9
- removed net TVIN3: CON1_GPIO-4.11
- removed net TVOUT0/VGA-G: CON1_GPIO-1.20
- removed net TVOUT1/VGA-B: CON1_GPIO-1.22
- removed net TVOUT2/VGA-R: CON1_GPIO-1.24
- removed net TVOUT3: CON1_GPIO-4.3
- removed net VMIC: CON1_GPIO-1.12
- removed net XN_TP: CON1_LCD.38
- removed net XP_TP: CON1_LCD.37
- removed net YN_TP: CON1_LCD.40
- removed net YP_TP: CON1_LCD.39
- new net N$47: RN7C.2, TP1.TP
- net CSI1_MLCK: now also TP2.TP
- net GND: now also JP1.1
